Commit message: Congigured joystick teleop, worked on navigation.

File: src/fenrir_description/urdf/fenrir.urdf.xacro (robot description, xacro)
@@ -190,5 +190,5 @@
     <parent link="base_link"/>
     <child link="lidar_link"/>
-    <origin xyz="0.1 0 0.05" rpy="0 0 0"/>
+    <origin xyz="0.0 0 0.0" rpy="0 0 0"/>
   </joint>
   <link name="lidar_link">
@@ -200,10 +200,4 @@
                izz="2.30279421279312E-08" />
     </inertial>
-    <collision>
-      <origin xyz= "0 0 0" rpy= "0 0 0"/>
-      <geometry>
-        <sphere radius= '0.05'/>
-      </geometry>
-    </collision>
   </link>
 </robot>

File: src/fenrir_description/urdf/fenrir_gazebo.xacro (robot description, xacro)
@@ -170,4 +170,5 @@
     <gazebo reference="lidar_link">
         <sensor type="gpu_lidar" name='lidar'>
+            <pose>0.0 0 0.0 0 0 0</pose>
             <frame_name>lidar_link</frame_name>
             <always_on>true</always_on>
